Commit message: 更新到最新版机械臂模型

File: src/arm/arm/model/robotic_arm.urdf (robot description, URDF)
Before this commit: robot robotic_arm, 8 links, 7 joints
Links:
- link base_link: mass 1.0998 -> 1.0608896790749
- link link1: mass 2.34956808405639 -> 1.3415964916658; geometry collision mesh filename=package://arm/model/Link1.STL; visual mesh filename=package://arm/model/Link1.STL
- link link2: mass 1.23727124080295 -> 1.1688360536306; geometry collision mesh filename=package://arm/model/Link2.STL; visual mesh filename=package://arm/model/Link2.STL
- link link3: mass 0.370266089775016 -> 0.697933163337346; geometry collision mesh filename=package://arm/model/Link3.STL; visual mesh filename=package://arm/model/Link3.STL
- link link4: mass 1.54177209165349 -> 0.37892648177412; geometry collision mesh filename=package://arm/model/Link4.STL; visual mesh filename=package://arm/model/Link4.STL
- link link5: mass 0.0698721570199944 -> 0.112337074738347; geometry collision mesh filename=package://arm/model/Link5.STL; visual mesh filename=package://arm/model/Link5.STL
- link link6: mass 0.128099358994803 -> 0.150213928644986; geometry collision mesh filename=package://arm/model/Link6.STL; visual mesh filename=package://arm/model/Link6.STL
Joints:
- joint joint1: axis 0 0 1 -> 0 0 -1; limit lower=-2.0 upper=2.0 effort=50 velocity=10 -> lower=-3.1 upper=3.1 effort=50 velocity=10; origin xyz=0 0 0 rpy=0 0 0 -> xyz=0 0 0.04875 rpy=0 0 0
- joint joint2: axis 0 0 1 -> 0 0 -1; limit lower=-1.570796327 upper=1.570796327 effort=50 velocity=10 -> lower=-1.57 upper=1.57 effort=50 velocity=10; origin xyz=0 0.03675 0.153 rpy=1.5708 -1.5708 0 -> xyz=0 -0.02575 0.08875 rpy=-1.5708 -1.5708 0
- joint joint3: origin xyz=0.52 0 0.08565 rpy=0 0 0 -> xyz=0.5 0 0.044 rpy=0 0 0
- joint joint4: axis 0 0 1 -> 0 0 -1; limit lower=-2.0 upper=1.8 effort=50 velocity=10 -> lower=-2 upper=2 effort=50 velocity=10; origin xyz=0.436 0 0.0225 rpy=0 0 0 -> xyz=0.49464 0 0.04645 rpy=0 0 0
- joint joint5: limit lower=-0.0349 upper=0.0349 effort=50 velocity=10 -> lower=-0.4 upper=0.4 effort=50 velocity=10; origin xyz=0.07761 -0.0058889 -0.03035 rpy=-1.5708 0 0 -> xyz=0.076 -0.044 -0.02455 rpy=-1.5708 0 0
- joint joint6: limit lower=-3.14159 upper=3.14159 effort=50 velocity=10 -> lower=0 upper=0 effort=50 velocity=10; origin xyz=0.073796 0.0036822 8.8922E-05 rpy=0 -1.5708 3.14 -> xyz=0.055 0 0.04675 rpy=-1.333 1.5708 -1.4022

Commit message: 抓取动作的更改

File: src/arm/arm/model/robotic_arm.urdf (robot description, URDF)
Before this commit: robot 质修R2仿制电科云台机械臂666URDF, 8 links, 7 joints
Joints:
- joint joint1: limit lower=-3.1 upper=3.1 effort=50 velocity=10 -> lower=-2.1 upper=2.1 effort=50 velocity=10
- joint joint5: axis 0 0 1 -> 0 0 -1

Commit message: 更新urdf

File: src/arm/arm/model/robotic_arm.urdf (robot description, URDF)
Before this commit: robot 质修R2仿制电科云台机械臂666URDF, 8 links, 7 joints
Links:
- link base_link: mass 1.0608896790749 -> 0.905716018714615
- link link1: mass 1.3415964916658 -> 1.91180538368796; geometry collision mesh filename=package://arm/model/link1.STL; visual mesh filename=package://arm/model/link1.STL
- link link2: mass 1.1688360536306 -> 1.09233144358037; geometry collision mesh filename=package://arm/model/link2.STL; visual mesh filename=package://arm/model/link2.STL
- link link3: mass 0.697933163337346 -> 0.750870225721497; geometry collision mesh filename=package://arm/model/link3.STL; visual mesh filename=package://arm/model/link3.STL
- link link4: mass 0.37892648177412 -> 0.328855136025888; geometry collision mesh filename=package://arm/model/link4.STL; visual mesh filename=package://arm/model/link4.STL
- link link5: mass 0.112337074738347 -> 0.107863966418761; geometry collision mesh filename=package://arm/model/link5.STL; visual mesh filename=package://arm/model/link5.STL
- link link6: mass 0.150213928644986 -> 0.150213928644987; geometry collision mesh filename=package://arm/model/link6.STL; visual mesh filename=package://arm/model/link6.STL
Joints:
- joint joint1: axis 0 0 -1 -> 0 0 1; limit lower=-2.1 upper=2.1 effort=50 velocity=10 -> lower=-3.14 upper=3.14 effort=50 velocity=10; origin xyz=0 0 0.04875 rpy=0 0 0 -> xyz=6.34132927793407E-05 -0.00167405073291106 0.0278500000000087 rpy=0 0 0; type revolute -> continuous
- joint joint2: origin xyz=0 -0.02575 0.08875 rpy=-1.5708 -1.5708 0 -> xyz=0.00565491862295636 0.0185517283813911 0.0710733482199691 rpy=-1.5707963267949 -1.5708 0
- joint joint3: axis 0 0 1 -> 0 0 -1; limit lower=-2.9 upper=2.9 effort=50 velocity=10 -> lower=-2.8 upper=2.8 effort=50 velocity=10; origin xyz=0.5 0 0.044 rpy=0 0 0 -> xyz=0.500001547205985 -0.00750000000003981 0.0418960557056171 rpy=3.14159265358979 0 0
- joint joint4: limit lower=-2 upper=2 effort=50 velocity=10 -> lower=-1.82 upper=1.92 effort=100 velocity=1; origin xyz=0.49464 0 0.04645 rpy=0 0 0 -> xyz=0.493372719987381 -0.000717203264851807 -0.0115 rpy=3.14159265358979 0 1.5708
- joint joint5: axis 0 0 -1 -> -0.0571545044239792 0 -0.998365345263972; origin xyz=0.076 -0.044 -0.02455 rpy=-1.5708 0 0 -> xyz=0.0420000017681742 0.0760000060786439 -0.0298499999999999 rpy=1.5707963267949 0 1.5708
- joint joint6: limit lower=0 upper=0 effort=50 velocity=10 -> lower=-3.14 upper=3.14 effort=50 velocity=10; origin xyz=0.055 0 0.04675 rpy=-1.333 1.5708 -1.4022 -> xyz=0.109242825291171 -0.00191951430536242 -0.0510772149208419 rpy=0.0171393597075962 1.51361065936655 3.14159265358978

Commit message: 更新新版机械臂位置之后

File: src/arm/arm/model/robotic_arm.urdf (robot description, URDF)
Before this commit: robot robotic_arm, 8 links, 7 joints
Joints:
- joint joint1: axis 0 0 1 -> 0 0 -1
- joint joint3: axis 0 0 -1 -> 0 0 1

Commit message: 提交1区抓取任务

File: src/arm/arm/model/robotic_arm.urdf (robot description, URDF)
Before this commit: robot robotic_arm, 8 links, 7 joints
Joints:
- joint joint3: axis 0 0 1 -> 0 0 -1
- joint joint5: axis -0.0571545044239792 0 -0.998365345263972 -> -0.0571545044239792 0 0.998365345263972
